Commit message: [modify]gps plugin

File: urdf/sam_bot_description.urdf.xacro (robot description, xacro)
@@ -145,4 +145,32 @@
       <pose>0 0 0 0 0 0</pose>
     </sensor>
+  </gazebo>
+  <link name="gps_link">
+    <visual>
+      <geometry>
+        <box size="0.1 0.1 0.1"/>
+      </geometry>
+    </visual>
+    <collision>
+      <geometry>
+        <box size="0.1 0.1 0.1"/>
+      </geometry>
+    </collision>
+    <xacro:box_inertia m="0.1" w="0.1" d="0.1" h="0.1"/>
+  </link>
+  <joint name="gps_joint" type="fixed">
+    <parent link="base_link"/>
+    <child link="gps_link"/>
+    <origin xyz="0 0 0.01"/>
+  </joint>
+  <gazebo>
+    <plugin name="gps" filename="libhector_gazebo_ros_gps.so">
+        <updateRate>10.0</updateRate>
+        <topicName>gps/fix</topicName>
+        <gaussianNoise>0.0 0.0 0.0</gaussianNoise>
+        <offset>0 0 0</offset>
+        <velocityGaussianNoise>0 0 0</velocityGaussianNoise>
+        <frameId>gps_link</frameId>
+    </plugin>
   </gazebo>
 <!--
